File: demos/stickhub/StickHub.kicad_sch (KiCad schematic)
At the start: 94 parts, among them J1 HOST, J2 USB1, J3 USB2, J4 USB3, J5 USB4, J6 USB5, J7 USB6, J8 USB7, J9 EXTGND, U1 MaxLinear_XR22417-48, U2 Dialog_SLG5NT1487V, Y1 12MHz 50ppm 16-20pF

Commit message: feat: add SPICE simulation module and related tests
- Implemented a new SPICE simulation module in `spice.py` that exports KiCad schematics to SPICE netlists and runs simulations using ngspice.
- Added preprocessing for netlists to handle power placeholders and GND mappings.
- Created tests for drawing an RC circuit, probing simulation symbols, and running SPICE simulations.
- Verified the integration of the `kicad_sch_simulate` tool within the MCP session.
Parts:
- added C1: 100n, symbol Device:C
- added LED1: Red, symbol Device:LED
- added R1 (x2): 10k, symbol Device:R
Other:
- note added: "Hello from MCP patched KiCad 10"
- note added: "MCP Demo: R1 + LED1"
