File: demos/keyboard-89/keyboard_matrix.kicad_sch (KiCad schematic)
At the start: 178 parts

Commit message: Add ERC report, AI setup documentation, and bootstrap scripts
- Created a new ERC report for the keyboard-89 project detailing isolated pin labels and library issues.
- Added AI environment bootstrap documentation for setting up the development environment on Windows and Linux.
- Implemented a PowerShell bootstrap script for Windows to automate the setup of dependencies, environment, and build process.
- Developed a corresponding bash bootstrap script for Linux with similar functionality.
- Introduced a new test for verifying pin connections in the symbol writer module.
- Added JSON report for failed drawing processes with a specific error message in Chinese.
Parts:
- TC-!1, TC-(1, TC-)1, TC-1, TC-10, TC-2, TC-3, TC-4, TC-5, TC-6, TC-7, TC-8, TC-9, TC-:;1, TC-@1, TC-A1, TC-B1, TC-C1, TC-D1, TC-E1, TC-F(0-9)1, TC-F1, TC-F2, TC-F3, TC-F4, TC-G1, TC-H1, TC-I1, TC-J1, TC-K1, TC-L1, TC-M1, TC-N1, TC-O1, TC-P1, TC-Q1, TC-R1, TC-S1, TC-T1, TC-U1, TC-V1, TC-W1, TC-X1, TC-Y1, TC-Z1, TC-\#1, TC-\$1, TC-\%1, TC-\&1, TC-\*-L1, TC-\*-R1, TC-\+1, TC-\+=1, TC-\-1, TC-\.1, TC-\/1, TC-\<,1, TC-\>.1, TC-^1, TC-`1, TC-alt1, TC-backspace1, TC-blankspace1, TC-bottom1, TC-capslock1, TC-ctrl1, TC-delete1, TC-end1, TC-enter-L1, TC-enter-R1, TC-esc1, TC-home1, TC-left1, TC-pagedown1, TC-pageup1, TC-printscreen1, TC-right1, TC-shift-L1, TC-shift-R1, TC-tab1, TC-top1, TC-windows1, TC-{[1, TC-|\1, TC-}]1, TC-—-1, TC-“‘1, TC-？/1, TC-～1: symbol private_lib:TC-6601-5-160G -> keyboard-89_local:TC-6601-5-160G
